File: v0.5/FrameworkGPU to MXM v0.5.kicad_pcb (KiCad board)
At the start: 4 copper layers, 109.6 x 64.7 mm, 119 parts, among them J1 MXM3.0, U2 FXBeam, U54 BR24G32FVT-3GE2

Commit message: Diff routed
Parts:
- removed R16: 220nF, TinkerForge:0603
- moved R22 0.61 mm to (67.4, 53.7)
- moved R9 0.41 mm to (85.3, 56.0)
- moved R30 0.40 mm to (76.3, 52.7)
- moved R10 0.40 mm to (83.7, 56.0)
- moved R26 0.32 mm to (70.4, 53.2)
- moved R1 0.30 mm to (71.2, 60.1)
- moved R23 0.30 mm to (68.4, 60.4)
- moved R20 0.22 mm to (64.5, 54.3)
- moved R3 0.22 mm to (72.6, 60.2)
- moved R2 0.22 mm to (74.5, 56.7)
- moved R4 0.22 mm to (73.0, 56.7)
- moved R7 0.22 mm to (77.0, 60.3)
- moved R25 0.22 mm to (71.9, 53.1), turned to 90 degrees
- moved R14 0.20 mm to (85.4, 60.2)
- moved R17 0.14 mm to (70.4, 56.6)
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Connections:
- J1 pad 11_13_15_17: GND -> (no net)
- J1 pad 1_3_5_7_9: +5V -> (no net)
- J1 pad 278_280: +3.3V -> (no net)
Routing:
- net PEX_RX7P: track 20.2 -> 44.6 mm, vias 0 -> 2
- net Net-(J1-PEX_RX7): track 23.3 -> 0.00 mm, vias 2 -> 0
- net PEX_TX4N: track 46.7 -> 60.2 mm
- net DP_A_L1P: track 77.4 -> 89.7 mm
- net PEX_TX1N: track 31.7 -> 40.9 mm
- net Net-(J1-PEX_TX7-): track 19.8 -> 28.3 mm
- net Net-(J1-PEX_RX0): track 23.1 -> 30.5 mm
- net PEX_TX2N: track 38.9 -> 45.5 mm
- net GND: track 258.6 -> 253.1 mm
- net Net-(J1-PEX_TX1-): track 5.17 -> 0.00 mm
- net PEX_TX5P: track 46.9 -> 51.7 mm
- net Net-(J1-PEX_TX4-): track 4.48 -> 0.00 mm
- net Net-(J1-PEX_TX5): track 4.16 -> 0.00 mm
- net Net-(J1-PEX_RX1): track 19.8 -> 23.8 mm
- net PEX_RX6P: track 11.0 -> 13.5 mm
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
Commit message: committing final version sent off for manufacturing
Parts:
- added C8: 220nF, TinkerForge:0603, F.Cu at (88.8, 56.4)
- R17, R18, R19, R20, R21, R22, R23, R24, R25, R26, R27, R28, R29, R30, R31, R32: value 10K -> 0
- moved TP22 49.6 mm to (91.7, 52.2)
- moved TP23 44.7 mm to (93.1, 67.7)
- moved R63 0.90 mm to (102.5, 59.3)
- turned R25 to -90 degrees
- turned R28 to -90 degrees
- renumbered R1 to C1, R2 to C10, R5 to C11, R7 to C12, R9 to C13, R11 to C14, R13 to C15, R15 to C16, R4 to C2, R6 to C3, R8 to C4, R10 to C5, R12 to C6, R14 to C7, R3 to C9
Connections:
- TP22 pad 1: SMB_DAT -> Net-(J1-SMB_DAT)
- TP23 pad 1: SMB_CLK -> Net-(J1-SMB_CLK)
- TP24 pad 1: TH_OVERT -> Net-(J1-TH_OVERT#)
- TP25 pad 1: TH_ALERT -> Net-(J1-TH_ALERT#)
- TP26 pad 1: TH_PWM -> Net-(J1-TH_PWM)
- TP27 pad 1: PWR_LEVEL -> Net-(J1-PWR_LEVEL)
- TP28 pad 1: PWR_GOOD -> Net-(J1-PWR_GOOD)
- TP29 pad 1: PWR_EN -> Net-(J1-PWR_EN)
Routing:
- net SMB_CLK: track 82.1 -> 46.6 mm, vias 3 -> 2
- net SMB_DAT: track 83.4 -> 49.1 mm, vias 3 -> 2
- net Net-(J1-TH_ALERT#): track 9.87 -> 34.7 mm, vias 0 -> 2
- net PEX_RX7P: track 44.6 -> 20.2 mm, vias 2 -> 0
- net Net-(J1-TH_OVERT#): track 6.65 -> 29.6 mm, vias 0 -> 2
- net GND: track 253.1 -> 275.9 mm, vias 73 -> 75
- net Net-(J1-PEX_RX7): track 0.00 -> 22.8 mm, vias 0 -> 2
- net TH_ALERT: track 51.8 -> 30.8 mm
- net Net-(J1-PWR_EN): track 6.32 -> 26.4 mm
- net (no net): track 19.9 -> 0.00 mm, vias 2 -> 0
- net Net-(J1-PWR_GOOD): track 9.74 -> 25.9 mm
- net Net-(J1-SMB_CLK): track 6.69 -> 21.1 mm, vias 0 -> 2
- net PWR_GOOD: track 62.5 -> 48.5 mm
- net Net-(J1-PWR_LEVEL): track 10.1 -> 22.6 mm
- net PWR_LEVEL: track 42.7 -> 31.9 mm
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- added copper zone on In3.Cu, net GND
- added copper zone on In4.Cu, net GND
Other:
- board size 109.6 x 64.7 mm -> 109.6 x 65.5 mm
- copper layers 4 -> 6
